Commit message: commit new

File: description/robot_core.xacro (robot description, xacro)
@@ -1,4 +1,16 @@
 <?xml version="1.0"?>
 <robot xmlns:xacro="http://www.ros.org/wiki/xacro">
+    <material name="white">
+        <color rgba="1 1 1 1"/>
+    </material>
+    <material name="orange">
+        <color rgba="1 0.3 0.1 1"/>
+    </material>
+    <material name="blue">
+        <color rgba="0.2 0.2 1 1"/>
+    </material>
+    <material name="black">
+        <color rgba="0 0 0 1"/>
+    </material>
     <link name="base_link">
     </link>
@@ -16,4 +28,12 @@
             <material name="white"/>
         </visual>
+        <collision>
+            <collision>
+                <origin xyz="0.15 0 0.075" rpy="0 0 0"/>
+                <geometry>
+                    <box size="0.3 0.3 0.15"/>
+                </geometry>
+            </collision>
+        </collision>
     </link>
     <!-- LEFT WHEEL -->
@@ -47,3 +67,17 @@
     </visual>
 </link>
+<!-- CASTER WHEEL -->
+<joint name="caster_wheel_joint" type="fixed">
+    <parent link="chassis"/>
+    <child link="caster_wheel"/>
+    <origin xyz="0.24 0 0" rpy="0 0 0"/>
+</joint>
+<link name="caster_wheel">
+    <visual>
+        <geometry>
+            <sphere radius="0.05" />
+        </geometry>
+        <material name="black"/>
+    </visual>
+</link>
 </robot>

Commit message: corrected collision properties

File: description/robot_core.xacro (robot description, xacro)
@@ -1,4 +1,5 @@
 <?xml version="1.0"?>
 <robot xmlns:xacro="http://www.ros.org/wiki/xacro">
+    <xacro:include filename="inertial_macros.xacro"/>
     <material name="white">
         <color rgba="1 1 1 1"/>
@@ -29,10 +30,8 @@
         </visual>
         <collision>
-            <collision>
                 <origin xyz="0.15 0 0.075" rpy="0 0 0"/>
                 <geometry>
                     <box size="0.3 0.3 0.15"/>
                 </geometry>
-            </collision>
         </collision>
     </link>
@@ -51,4 +50,10 @@
         <material name="blue"/>
     </visual>
+    <collision>
+        <geometry>
+            <cylinder length="0.04" radius="0.05" />
+        </geometry>
+        <material name="blue"/>
+    </collision>
 </link>
 <!-- RIGHT WHEEL -->
@@ -66,4 +71,10 @@
         <material name="blue"/>
     </visual>
+    <collision>
+        <geometry>
+            <cylinder length="0.04" radius="0.05" />
+        </geometry>
+        <material name="blue"/>
+    </collision>
 </link>
 <!-- CASTER WHEEL -->
@@ -80,4 +91,10 @@
         <material name="black"/>
     </visual>
+    <collision>
+        <geometry>
+            <sphere radius="0.05" />
+        </geometry>
+        <material name="black"/>
+    </collision>
 </link>
 </robot>

Commit message: removed collision elements

File: description/robot_core.xacro (robot description, xacro)
@@ -29,10 +29,4 @@
             <material name="white"/>
         </visual>
-        <collision>
-                <origin xyz="0.15 0 0.075" rpy="0 0 0"/>
-                <geometry>
-                    <box size="0.3 0.3 0.15"/>
-                </geometry>
-        </collision>
     </link>
     <!-- LEFT WHEEL -->

Commit message: final commit

File: description/robot_core.xacro (robot description, xacro)
@@ -2,4 +2,7 @@
 <robot xmlns:xacro="http://www.ros.org/wiki/xacro">
     <xacro:include filename="inertial_macros.xacro"/>
+    <xacro:include filename="gazebo_control.xacro"/>
+    <xacro:include filename="lidar.xacro" />
+    <xacro:include filename="camera.xacro" />
     <material name="white">
         <color rgba="1 1 1 1"/>
@@ -13,4 +16,7 @@
     <material name="black">
         <color rgba="0 0 0 1"/>
+    </material>
+    <material name="red">
+        <color rgba="1 0 0 1"/>
     </material>
     <link name="base_link">
